Commit message: diff robot

File: src/description_bauda_mec/description/base.urdf.xacro (robot description, xacro)
@@ -42,4 +42,7 @@
         </xacro:inertial_box>
     </link>
+    <gazebo reference="chassis">
+        <material>Gazebo/White</material>
+    </gazebo>
     <!-- Left front wheel -->
     <joint name="lf_wheel_joint" type="continuous">
@@ -65,4 +68,7 @@
         </xacro:inertial_cylinder>
     </link>
+    <gazebo reference="lf_wheel">
+        <material>Gazebo/Red</material>
+    </gazebo>
     <!-- Right front wheel -->
     <joint name="rf_wheel_joint" type="continuous">
@@ -88,4 +94,7 @@
         </xacro:inertial_cylinder>
     </link>
+    <gazebo reference="rf_wheel">
+        <material>Gazebo/Red</material>
+    </gazebo>
     <!-- Left rear wheel -->
     <joint name="lr_wheel_joint" type="continuous">
@@ -111,4 +120,7 @@
         </xacro:inertial_cylinder>
     </link>
+    <gazebo reference="lr_wheel">
+        <material>Gazebo/Red</material>
+    </gazebo>
     <!-- Right rear wheel -->
     <joint name="rr_wheel_joint" type="continuous">
@@ -134,3 +146,6 @@
         </xacro:inertial_cylinder>
     </link>
+    <gazebo reference="rr_wheel">
+        <material>Gazebo/Red</material>
+    </gazebo>
 </robot>

File: src/description_bauda_mec/description/robot.urdf.xacro (robot description, xacro)
@@ -1,4 +1,5 @@
 <?xml version="1.0"?>
 <robot xmlns:xacro="http://www.ros.org/wiki/xacro"  name="bauda_mec">
-    <xacro:include filename="$(find description_bauda_akm)/description/base.urdf.xacro" />
+    <xacro:include filename="$(find description_bauda_mec)/description/base.urdf.xacro" />
+    <xacro:include filename="$(find description_bauda_mec)/description/gazebo_control.xacro"/>
 </robot>
