Commit message: Tentativa de controle akm gazebo

File: src/description_bauda_akm/description/gazebo_control.xacro (robot description, xacro)
@@ -1,20 +1,45 @@
 <?xml version="1.0"?>
 <robot xmlns:xacro="http://www.ros.org/wiki/xacro">
+    <xacro:property name="yaml_file" value="$(find description_bauda_akm)/config/vehicle.yaml" />
+    <xacro:property name="vehicle_dict" value="${load_yaml(yaml_file)}"/>
+    <xacro:property name="steering_limit_angle" value="${vehicle_dict['steering']['limit_angle']}" />
     <gazebo>
-        <plugin name="diff_drive" filename="libgazebo_ros_diff_drive.so">
-            <!-- Wheel Information -->
-            <left_joint>left_wheel_joint</left_joint>
-            <right_joint>right_wheel_joint</right_joint>
-            <wheel_separation>0.35</wheel_separation>
-            <wheel_diameter>0.1</wheel_diameter>
-            <!-- Limits -->
-            <max_wheel_torque>200</max_wheel_torque>
-            <max_wheel_acceleration>10.0</max_wheel_acceleration>
-            <!-- Output -->
-            <odometry_frame>odom</odometry_frame>
-            <robot_base_frame>base_link</robot_base_frame>
+        <plugin name="ackermann_drive" filename="libgazebo_ros_ackermann_drive.so">
+            <!-- <ros>
+                <namespace>demo</namespace>
+                <remapping>cmd_vel:=cmd_demo</remapping>
+                <remapping>odom:=odom_demo</remapping>
+                <remapping>distance:=distance_demo</remapping>
+            </ros> -->
+            <update_rate>100.0</update_rate>
+            <!-- wheels -->
+            <front_left_joint>front_left_wheel_joint</front_left_joint>
+            <front_right_joint>front_right_wheel_joint</front_right_joint>
+            <rear_left_joint>rear_left_wheel_joint</rear_left_joint>
+            <rear_right_joint>rear_right_wheel_joint</rear_right_joint>
+            <left_steering_joint>left_steering_joint</left_steering_joint>
+            <right_steering_joint>right_steering_joint</right_steering_joint>
+            <steering_wheel_joint>steering_wheel_joint</steering_wheel_joint>
+            <!-- Max absolute steer angle for tyre in radians-->
+            <!-- Any cmd_vel angular z greater than this would be capped -->
+            <max_steer>${steering_limit_angle}</max_steer>
+            <!-- Max absolute steering angle of steering wheel -->
+            <max_steering_angle>9.42</max_steering_angle>
+            <!-- Max absolute linear speed in m/s -->
+            <max_speed>20</max_speed>
+            <!-- PID tuning -->
+            <left_steering_pid_gain>1500 0 1</left_steering_pid_gain>
+            <left_steering_i_range>0 0</left_steering_i_range>
+            <right_steering_pid_gain>1500 0 1</right_steering_pid_gain>
+            <right_steering_i_range>0 0</right_steering_i_range>
+            <linear_velocity_pid_gain>1000 0 1</linear_velocity_pid_gain>
+            <linear_velocity_i_range>0 0</linear_velocity_i_range>
+            <!-- output -->
             <publish_odom>true</publish_odom>
             <publish_odom_tf>true</publish_odom_tf>
             <publish_wheel_tf>true</publish_wheel_tf>
+            <publish_distance>true</publish_distance>
+            <odometry_frame>odom_demo</odometry_frame>
+            <robot_base_frame>base_link</robot_base_frame>
         </plugin>
     </gazebo>

File: src/description_bauda_akm/description/robot.urdf.xacro (robot description, xacro)
@@ -2,3 +2,4 @@
 <robot xmlns:xacro="http://www.ros.org/wiki/xacro"  name="bauda_diff">
     <xacro:include filename="robot_core.xacro" />
+    <xacro:include filename="gazebo_control.xacro" />
 </robot>

File: src/description_bauda_akm/description/robot_core.xacro (robot description, xacro)
@@ -21,5 +21,5 @@
     <!-- BASE LINK -->
     <link name="base_link" />
-    <!-- BASE_FOOTPRINT LINK -->
+    <!-- BASE_FOOTPRINT -->
     <joint name="base_footprint_joint" type="fixed">
         <parent link="base_link"/>
@@ -28,5 +28,5 @@
     </joint>
     <link name="base_footprint" />
-    <!-- CHASSIS LINK -->
+    <!-- CHASSIS -->
     <joint name="chassis_joint" type="fixed">
         <parent link="base_link"/>
@@ -55,5 +55,5 @@
         <material>Gazebo/White</material>
     </gazebo>
-    <!-- REAR LEFT WHEEL LINK -->
+    <!-- REAR LEFT WHEEL -->
     <joint name="rear_left_wheel_joint" type="continuous">
         <parent link="base_link"/>
@@ -81,5 +81,5 @@
         <material>Gazebo/Blue</material>
     </gazebo>
-    <!-- REAR RIGHT WHEEL LINK -->
+    <!-- REAR RIGHT WHEEL -->
     <joint name="rear_right_wheel_joint" type="continuous">
         <parent link="base_link"/>
@@ -108,5 +108,5 @@
     </gazebo>
     <!-- LEFT STEERING -->
-    <joint name="left_steering" type="revolute">
+    <joint name="left_steering_joint" type="revolute">
         <parent link="base_link"/>
         <child link="left_steering_link"/>
@@ -116,7 +116,25 @@
                 effort="${steering_limit_effort}" velocity="${steering_limit_velocity}"/>
     </joint>
-    <link name="left_steering_link" />
+    <link name="left_steering_link">
+        <!-- <visual>
+            <geometry>
+                <cylinder radius="0.001" length="0.001"/>
+            </geometry>
+            <material name="blue"/>
+        </visual>
+        <collision>
+            <geometry>
+                <cylinder radius="0.001" length="0.001"/>
+            </geometry>
+        </collision>
+        <xacro:inertial_cylinder mass="0.001" length="0.001" radius="0.001">
+            <origin xyz="0 0 0" rpy="0 0 0"/>
+        </xacro:inertial_cylinder> -->
+    </link>
+    <!-- <gazebo reference="rear_right_wheel">
+        <material>Gazebo/Blue</material>
+    </gazebo> -->
     <!-- RIGHT STEERING -->
-    <joint name="right_steering" type="revolute">
+    <joint name="right_steering_joint" type="revolute">
         <parent link="base_link"/>
         <child link="right_steering_link"/>
@@ -126,6 +144,24 @@
                 effort="${steering_limit_effort}" velocity="${steering_limit_velocity}"/>
     </joint>
-    <link name="right_steering_link" />
-    <!-- FRONT LEFT WHEEL LINK -->
+    <link name="right_steering_link">
+        <!-- <visual>
+            <geometry>
+                <cylinder radius="0.001" length="0.001"/>
+            </geometry>
+            <material name="blue"/>
+        </visual>
+        <collision>
+            <geometry>
+                <cylinder radius="0.001" length="0.001"/>
+            </geometry>
+        </collision>
+        <xacro:inertial_cylinder mass="0.001" length="0.001" radius="0.001">
+            <origin xyz="0 0 0" rpy="0 0 0"/>
+        </xacro:inertial_cylinder> -->
+    </link>
+    <!-- <gazebo reference="rear_right_wheel">
+        <material>Gazebo/Blue</material>
+    </gazebo> -->
+    <!-- FRONT LEFT WHEEL -->
     <joint name="front_left_wheel_joint" type="continuous">
         <parent link="left_steering_link"/>
@@ -153,5 +189,5 @@
         <material>Gazebo/Blue</material>
     </gazebo>
-    <!-- FRONT RIGHT WHEEL LINK -->
+    <!-- FRONT RIGHT WHEEL -->
     <joint name="front_right_wheel_joint" type="continuous">
         <parent link="right_steering_link"/>
@@ -179,3 +215,29 @@
         <material>Gazebo/Blue</material>
     </gazebo>
+    <!-- STEERING WHEEL -->
+    <joint name="steering_wheel_joint" type="continuous">
+        <parent link="base_link"/>
+        <child link="steering_wheel"/>
+        <origin xyz="0 0 0" rpy="0 0 0"/>
+        <axis xyz="0 0 1"/>
+    </joint>
+    <link name="steering_wheel">
+        <!-- <visual>
+            <geometry>
+                <cylinder radius="${wheel_radius}" length="${wheel_width}"/>
+            </geometry>
+            <material name="blue"/>
+        </visual>
+        <collision>
+            <geometry>
+                <cylinder radius="${wheel_radius}" length="${wheel_width}"/>
+            </geometry>
+        </collision>
+        <xacro:inertial_cylinder mass="${wheel_mass}" length="${wheel_width}" radius="${wheel_radius}">
+            <origin xyz="0 0 0" rpy="0 0 0"/>
+        </xacro:inertial_cylinder> -->
+    </link>
+    <!-- <gazebo reference="front_right_wheel">
+        <material>Gazebo/Blue</material>
+    </gazebo> -->
  </robot>

File: src/description_bauda_akm/description/ros2_control.xacro (robot description, xacro)
@@ -1,9 +1,10 @@
 <?xml version="1.0"?>
 <robot xmlns:xacro="http://www.ros.org/wiki/xacro">
+    <xacro:property name="steering_limit_angle" value="${vehicle_dict['steering']['limit_angle']}" />
     <ros2_control name="GazeboSystem" type="system">
         <hardware>
             <plugin>gazebo_ros2_control/GazeboSystem</plugin>
         </hardware>
-        <joint name="left_wheel_joint">
+        <joint name="rear_left_wheel_joint">
             <command_interface name="velocity">
                 <param name="min">-10</param>
@@ -11,7 +12,6 @@
             </command_interface>
             <state_interface name="velocity"/>
-            <state_interface name="position"/>
         </joint>
-        <joint name="right_wheel_joint">
+        <joint name="rear_right_wheel_joint">
             <command_interface name="velocity">
                 <param name="min">-10</param>
@@ -19,4 +19,38 @@
             </command_interface>
             <state_interface name="velocity"/>
+        </joint>
+        <joint name="front_left_wheel_joint">
+            <command_interface name="velocity">
+                <param name="min">-10</param>
+                <param name="max">10</param>
+            </command_interface>
+            <state_interface name="velocity"/>
+        </joint>
+        <joint name="front_right_wheel_joint">
+            <command_interface name="velocity">
+                <param name="min">-10</param>
+                <param name="max">10</param>
+            </command_interface>
+            <state_interface name="velocity"/>
+        </joint>
+        <joint name="left_steering_joint">
+            <command_interface name="position">
+                <param name="min">${-steering_limit_angle}</param>
+                <param name="max">${steering_limit_angle}</param>
+            </command_interface>
+            <state_interface name="position"/>
+        </joint>
+        <joint name="right_steering_joint">
+            <command_interface name="position">
+                <param name="min">${-steering_limit_angle}</param>
+                <param name="max">${steering_limit_angle}</param>
+            </command_interface>
+            <state_interface name="position"/>
+        </joint>
+        <joint name="steering_wheel_joint">
+            <command_interface name="position">
+                <param name="min">${-steering_limit_angle}</param>
+                <param name="max">${steering_limit_angle}</param>
+            </command_interface>
             <state_interface name="position"/>
         </joint>
@@ -24,5 +58,5 @@
     <gazebo>
         <plugin name="gazebo_ros2_control" filename="libgazebo_ros2_control.so">
-            <parameters>$(find description_bauda_diff)/config/controllers.yaml</parameters>
+            <parameters>$(find description_bauda_akm)/config/controllers.yaml</parameters>
         </plugin>
     </gazebo>

Commit message: There isn't ackermann controller for foxy

File: src/description_bauda_akm/description/gazebo_control.xacro (robot description, xacro)
@@ -1,7 +1,7 @@
 <?xml version="1.0"?>
 <robot xmlns:xacro="http://www.ros.org/wiki/xacro">
-    <xacro:property name="yaml_file" value="$(find description_bauda_akm)/config/vehicle.yaml" />
+    <!-- <xacro:property name="yaml_file" value="$(find description_bauda_akm)/config/vehicle.yaml" />
     <xacro:property name="vehicle_dict" value="${load_yaml(yaml_file)}"/>
-    <xacro:property name="steering_limit_angle" value="${vehicle_dict['steering']['limit_angle']}" />
+    <xacro:property name="steering_limit_angle" value="${vehicle_dict['steering']['limit_angle']}" />  -->
     <gazebo>
         <plugin name="ackermann_drive" filename="libgazebo_ros_ackermann_drive.so">
@@ -23,5 +23,6 @@
             <!-- Max absolute steer angle for tyre in radians-->
             <!-- Any cmd_vel angular z greater than this would be capped -->
-            <max_steer>${steering_limit_angle}</max_steer>
+            <!-- <max_steer>${steering_limit_angle}</max_steer> -->
+            <max_steer>3.0</max_steer>
             <!-- Max absolute steering angle of steering wheel -->
             <max_steering_angle>9.42</max_steering_angle>
@@ -29,10 +30,10 @@
             <max_speed>20</max_speed>
             <!-- PID tuning -->
-            <left_steering_pid_gain>1500 0 1</left_steering_pid_gain>
+            <!-- <left_steering_pid_gain>1500 0 1</left_steering_pid_gain>
             <left_steering_i_range>0 0</left_steering_i_range>
             <right_steering_pid_gain>1500 0 1</right_steering_pid_gain>
             <right_steering_i_range>0 0</right_steering_i_range>
             <linear_velocity_pid_gain>1000 0 1</linear_velocity_pid_gain>
-            <linear_velocity_i_range>0 0</linear_velocity_i_range>
+            <linear_velocity_i_range>0 0</linear_velocity_i_range> -->
             <!-- output -->
             <publish_odom>true</publish_odom>
@@ -40,6 +41,6 @@
             <publish_wheel_tf>true</publish_wheel_tf>
             <publish_distance>true</publish_distance>
-            <odometry_frame>odom_demo</odometry_frame>
-            <robot_base_frame>base_link</robot_base_frame>
+            <!-- <odometry_frame>odom_demo</odometry_frame>
+            <robot_base_frame>base_link</robot_base_frame> -->
         </plugin>
     </gazebo>

File: src/description_bauda_akm/description/robot.urdf.xacro (robot description, xacro)
@@ -2,4 +2,5 @@
 <robot xmlns:xacro="http://www.ros.org/wiki/xacro"  name="bauda_diff">
     <xacro:include filename="robot_core.xacro" />
-    <xacro:include filename="gazebo_control.xacro" />
+    <!-- <xacro:include filename="gazebo_control.xacro" /> -->
+    <xacro:include filename="ros2_control.xacro" />
 </robot>

File: src/description_bauda_akm/description/robot_core.xacro (robot description, xacro)
@@ -117,4 +117,9 @@
     </joint>
     <link name="left_steering_link">
+        <inertial>
+            <origin xyz="0 0 0" rpy="0 0 0"/>
+            <mass value="0.02"/>
+            <inertia ixx="0.002" ixy="0" ixz="0" iyy="0.002" iyz="0" izz="0.002"/>
+        </inertial>
         <!-- <visual>
             <geometry>
@@ -145,4 +150,9 @@
     </joint>
     <link name="right_steering_link">
+        <inertial>
+            <origin xyz="0 0 0" rpy="0 0 0"/>
+            <mass value="0.02"/>
+            <inertia ixx="0.002" ixy="0" ixz="0" iyy="0.002" iyz="0" izz="0.002"/>
+        </inertial>
         <!-- <visual>
             <geometry>
@@ -219,25 +229,25 @@
         <parent link="base_link"/>
         <child link="steering_wheel"/>
-        <origin xyz="0 0 0" rpy="0 0 0"/>
+        <origin xyz="${wheel_distance_between_axes} 0 ${base_height + 2 * wheel_radius}" rpy="0 0 0"/>
         <axis xyz="0 0 1"/>
     </joint>
     <link name="steering_wheel">
-        <!-- <visual>
-            <geometry>
-                <cylinder radius="${wheel_radius}" length="${wheel_width}"/>
-            </geometry>
-            <material name="blue"/>
-        </visual>
-        <collision>
-            <geometry>
-                <cylinder radius="${wheel_radius}" length="${wheel_width}"/>
-            </geometry>
-        </collision>
-        <xacro:inertial_cylinder mass="${wheel_mass}" length="${wheel_width}" radius="${wheel_radius}">
-            <origin xyz="0 0 0" rpy="0 0 0"/>
-        </xacro:inertial_cylinder> -->
-    </link>
-    <!-- <gazebo reference="front_right_wheel">
-        <material>Gazebo/Blue</material>
-    </gazebo> -->
+        <visual>
+            <geometry>
+                <cylinder radius="${wheel_radius}" length="${wheel_width}"/>
+            </geometry>
+            <material name="blue"/>
+        </visual>
+        <collision>
+            <geometry>
+                <cylinder radius="${wheel_radius}" length="${wheel_width}"/>
+            </geometry>
+        </collision>
+        <xacro:inertial_cylinder mass="${wheel_mass}" length="${wheel_width}" radius="${wheel_radius}">
+            <origin xyz="0 0 0" rpy="0 0 0"/>
+        </xacro:inertial_cylinder>
+    </link>
+    <gazebo reference="steering_wheel">
+        <material>Gazebo/Blue</material>
+    </gazebo>
  </robot>
