Commit message: akm xacro

File: src/description_bauda_akm/description/robot.urdf.xacro (robot description, xacro)
@@ -2,8 +2,3 @@
 <robot xmlns:xacro="http://www.ros.org/wiki/xacro"  name="bauda_diff">
     <xacro:include filename="robot_core.xacro" />
-    <!-- <xacro:include filename="gazebo_control.xacro" /> -->
-    <xacro:include filename="ros2_control.xacro" />
-    <xacro:include filename="2D_lidar.xacro" />
-    <!-- <xacro:include filename="camera.xacro" /> -->
-    <xacro:include filename="depth_camera.xacro" />
 </robot>

File: src/description_bauda_akm/description/robot_core.xacro (robot description, xacro)
@@ -4,12 +4,14 @@
     <xacro:include filename="materials.xacro"/>
     <!-- Define robot constants https://navigation.ros.org/setup_guides/urdf/setup_urdf.html -->
+    <xacro:property name="yaml_file" value="$(find description_bauda_akm)/config/vehicle.yaml" />
+    <xacro:property name="dict" value="${load_yaml(yaml_file)}"/>
     <xacro:property name="base_mass" value="${dict['base'][mass]}" />
+    <xacro:property name="base_length" value="${dict['base'][length]}" />
     <xacro:property name="base_width" value="${dict['base'][width]}" />
-    <xacro:property name="base_length" value="${dict['base'][length]}" />
+    <xacro:property name="base_height" value="${dict['base'][height]}" />
     <xacro:property name="wheel_mass" value="${dict['wheel'][mass]}" />
     <xacro:property name="wheel_radius" value="${dict['wheel'][radius]}" />
     <xacro:property name="wheel_width" value="${dict['wheel'][width]}" />
     <xacro:property name="wheel_ygap" value="${dict['wheel'][ygap]}" />
-    <xacro:property name="wheel_zoff" value="${dict['wheel'][zoff]}" />
     <xacro:property name="wheel_rear_xoff" value="${dict['wheel'][rear_xoff]}" />
     <xacro:property name="wheel_front_xoff" value="${dict['wheel'][front_xoff]}" />
@@ -27,22 +29,22 @@
         <parent link="base_link"/>
         <child link="chassis"/>
-        <origin xyz="-0.1 0 0"/>
+        <origin xyz="-${wheel_rear_xoff} 0 0"/>
     </joint>
     <link name="chassis">
         <visual>
-            <origin xyz="0.15 0 0.075"/>
+            <origin xyz="${base_length / 2} 0 ${base_height / 2}"/>
             <geometry>
-                <box size="0.3 0.3 0.15"/>
+                <box size="${base_length} ${base_width} ${base_height}"/>
             </geometry>
             <material name="white"/>
         </visual>
         <collision>
-            <origin xyz="0.15 0 0.075"/>
+            <origin xyz="${base_length / 2} 0 ${base_height / 2}"/>
             <geometry>
-                <box size="0.3 0.3 0.15"/>
+                <box size="${base_length} ${base_width} ${base_height}"/>
             </geometry>
         </collision>
-        <xacro:inertial_box mass="0.5" x="0.3" y="0.3" z="0.15">
-            <origin xyz="0.15 0 0.075" rpy="0 0 0"/>
+        <xacro:inertial_box mass="${base_mass}" x="${base_length}" y="${base_width}" z="${base_height}">
+            <origin xyz="${base_length / 2} 0 ${base_height / 2}" rpy="0 0 0"/>
         </xacro:inertial_box>
     </link>
@@ -50,82 +52,3 @@
         <material>Gazebo/White</material>
     </gazebo>
-    <!-- LEFT WHEEL LINK -->
-    <joint name="left_wheel_joint" type="continuous">
-        <parent link="base_link"/>
-        <child link="left_wheel"/>
-        <origin xyz="0 0.175 0" rpy="-${pi/2} 0 0" />
-        <axis xyz="0 0 1"/>
-    </joint>
-    <link name="left_wheel">
-        <visual>
-            <geometry>
-                <cylinder radius="0.05" length="0.04"/>
-            </geometry>
-            <material name="blue"/>
-        </visual>
-        <collision>
-            <geometry>
-                <cylinder radius="0.05" length="0.04"/>
-            </geometry>
-        </collision>
-        <xacro:inertial_cylinder mass="0.1" length="0.04" radius="0.05">
-            <origin xyz="0 0 0" rpy="0 0 0"/>
-        </xacro:inertial_cylinder>
-    </link>
-    <gazebo reference="left_wheel">
-        <material>Gazebo/Blue</material>
-    </gazebo>
-    <!-- RIGHT WHEEL LINK -->
-    <joint name="right_wheel_joint" type="continuous">
-        <parent link="base_link"/>
-        <child link="right_wheel"/>
-        <origin xyz="0 -0.175 0" rpy="${pi/2} 0 0" />
-        <axis xyz="0 0 -1"/>
-    </joint>
-    <link name="right_wheel">
-        <visual>
-            <geometry>
-                <cylinder radius="0.05" length="0.04"/>
-            </geometry>
-            <material name="blue"/>
-        </visual>
-        <collision>
-            <geometry>
-                <cylinder radius="0.05" length="0.04"/>
-            </geometry>
-        </collision>
-        <xacro:inertial_cylinder mass="0.1" length="0.04" radius="0.05">
-            <origin xyz="0 0 0" rpy="0 0 0"/>
-        </xacro:inertial_cylinder>
-    </link>
-    <gazebo reference="right_wheel">
-        <material>Gazebo/Blue</material>
-    </gazebo>
-    <!-- CASTER WHEEL LINK -->
-    <joint name="caster_wheel_joint" type="fixed">
-        <parent link="chassis"/>
-        <child link="caster_wheel"/>
-        <origin xyz="0.24 0 0"/>
-    </joint>
-    <link name="caster_wheel">
-        <visual>
-            <geometry>
-                <sphere radius="0.05"/>
-            </geometry>
-            <material name="black"/>
-        </visual>
-        <collision>
-            <geometry>
-                <sphere radius="0.05"/>
-            </geometry>
-        </collision>
-        <xacro:inertial_sphere mass="0.1" radius="0.05">
-            <origin xyz="0 0 0" rpy="0 0 0"/>
-        </xacro:inertial_sphere>
-    </link>
-    <gazebo reference="caster_wheel">
-        <material>Gazebo/Black</material>
-        <mu1 value="0.001"/>
-        <mu2 value="0.001"/>
-    </gazebo>
 </robot>

File: src/description_bauda_akm/description/wheel.xacro (robot description, xacro)
@@ -1,296 +1,73 @@
 <?xml version="1.0"?>
 <robot name="wheel" xmlns:xacro="http://wiki.ros.org/xacro">
-  <xacro:include filename="materials.xacro"/>
-  <xacro:include filename="inertials.xacro"/>
-  <!-- Properties -->
-  <xacro:property name="steer_effort" value="10.0"/>
-  <xacro:property name="steer_velocity" value="5.0"/>
-  <xacro:property name="steer_limit_deg" value="45.0"/>
-  <!-- Bicycle model front steering link (required for steer_drive_controller) -->
-  <xacro:macro name="front_steer"
-    params="
-      name
-      parent
-      steer_radius
-      steer_thickness
-      steer_mass
-      base_length
-      base_width
-      axle_offset
-      steer_height">
-    <link name="${name}_steer_link">
-      <visual>
+    <xacro:include filename="materials.xacro"/>
+    <xacro:include filename="inertials.xacro"/>
+    <xacro:macro name="wheel" params="left_or_right rear_or_front">
+    <joint name="${rear_or_front}_${left_or_right}_wheel_joint" type="continuous">
+        <parent link="base_link"/>
+        <child link="${rear_or_front}_${left_or_right}_wheel"/>
+        <origin xyz="0 0.175 0" rpy="-${pi/2} 0 0" />
+        <axis xyz="0 0 1"/>
+    </joint>
+    <link name="left_wheel">
+        <visual>
+            <geometry>
+                <cylinder radius="0.05" length="0.04"/>
+            </geometry>
+            <material name="blue"/>
+        </visual>
+        <collision>
+            <geometry>
+                <cylinder radius="0.05" length="0.04"/>
+            </geometry>
+        </collision>
+        <xacro:inertial_cylinder mass="0.1" length="0.04" radius="0.05">
+            <origin xyz="0 0 0" rpy="0 0 0"/>
+        </xacro:inertial_cylinder>
+    </link>
+    <gazebo reference="left_wheel">
+        <material>Gazebo/Blue</material>
+    </gazebo>
+    <link name="${rear_or_front}_${left_or_right}_wheel_link">
+        <visual>
         <origin xyz="0 0 0" rpy="0 0 0"/>
         <geometry>
-          <cylinder radius="${steer_radius}" length="${steer_thickness}"/>
+            <cylinder radius="${steer_radius}" length="${steer_thickness}"/>
         </geometry>
         <material name="yellow" />
-      </visual>
-      <collision>
+        </visual>
+        <collision>
         <origin xyz="0 0 0" rpy="0 0 0"/>
         <geometry>
-          <cylinder radius="${steer_radius}" length="${steer_thickness}"/>
+            <cylinder radius="${steer_radius}" length="${steer_thickness}"/>
         </geometry>
-      </collision>
-      <xacro:solid_cylinder_inertial
-          rpy="0 0 0" xyz="0 0 0"
-          mass="${steer_mass}"
-          radius="${steer_radius}" length="${steer_thickness}" />
+        </collision>
+        <xacro:solid_cylinder_inertial
+            rpy="0 0 0" xyz="0 0 0"
+            mass="${steer_mass}"
+            radius="${steer_radius}" length="${steer_thickness}" />
     </link>
     <joint name="${name}_steer_joint" type="revolute">
-      <parent link="${parent}_link"/>
-      <child link="${name}_steer_link"/>
-      <origin xyz="${base_length/2-axle_offset} 0 ${steer_height}" rpy="0 0 0"/>
-      <axis xyz="0 0 1"/>
-      <limit effort="${steer_effort}"
-             lower="${-180.0 * deg_to_rad}" upper="${180.0 * deg_to_rad}"
-             velocity="${steer_velocity}"/>
+        <parent link="${parent}_link"/>
+        <child link="${name}_steer_link"/>
+        <origin xyz="${base_length/2-axle_offset} 0 ${steer_height}" rpy="0 0 0"/>
+        <axis xyz="0 0 1"/>
+        <limit effort="${steer_effort}"
+                lower="${-180.0 * deg_to_rad}" upper="${180.0 * deg_to_rad}"
+                velocity="${steer_velocity}"/>
     </joint>
     <transmission name="${name}_steer_joint_trans">
-      <type>transmission_interface/SimpleTransmission</type>
-      <actuator name="${name}_steer_joint_motor">
+        <type>transmission_interface/SimpleTransmission</type>
+        <actuator name="${name}_steer_joint_motor">
         <mechanicalReduction>1</mechanicalReduction>
         <hardwareInterface>hardware_interface/PositionJointInterface</hardwareInterface>
-      </actuator>
-      <joint name="${name}_steer_joint">
+        </actuator>
+        <joint name="${name}_steer_joint">
         <hardwareInterface>hardware_interface/PositionJointInterface</hardwareInterface>
-      </joint>
+        </joint>
     </transmission>
     <gazebo reference="${name}_steer_link">
-      <material>Gazebo/Yellow</material>
+        <material>Gazebo/Yellow</material>
     </gazebo>
-  </xacro:macro>
-  <!-- Car steering model front (steerable) wheel links (left/right) -->
-  <xacro:macro name="front_wheel_lr"
-    params="
-      name
-      parent
-      reflect
-      wheel_radius
-      wheel_thickness
-      wheel_mass
-      steer_radius
-      steer_thickness
-      steer_mass
-      base_length
-      base_width
-      axle_offset
-      steer_height">
-    <link name="${name}_steer_link">
-      <visual>
-        <origin xyz="0 0 0" rpy="0 0 0"/>
-        <geometry>
-          <cylinder radius="${steer_radius}" length="${steer_thickness}"/>
-        </geometry>
-        <material name="blue" />
-      </visual>
-      <collision>
-        <origin xyz="0 0 0" rpy="0 0 0"/>
-        <geometry>
-          <cylinder radius="${steer_radius}" length="${steer_thickness}"/>
-        </geometry>
-      </collision>
-      <xacro:solid_cylinder_inertial
-          rpy="0 0 0" xyz="0 0 0"
-          mass="${steer_mass}"
-          radius="${steer_radius}" length="${steer_thickness}" />
-    </link>
-    <joint name="${name}_steer_joint" type="revolute">
-      <parent link="${parent}_link"/>
-      <child link="${name}_steer_link"/>
-      <origin xyz="${base_length/2-axle_offset} ${reflect*(base_width/2+axle_offset)} ${steer_height}" rpy="0 0 0"/>
-      <axis xyz="0 0 1"/>
-      <limit effort="${steer_effort}"
-             lower="${steer_limit_deg * deg_to_rad * -1.0}" upper="${steer_limit_deg * deg_to_rad}"
-             velocity="${steer_velocity}"/>
-    </joint>
-    <link name="${name}_wheel_link">
-      <visual>
-        <origin xyz="0 0 0" rpy="0 0 0"/>
-        <geometry>
-          <cylinder radius="${wheel_radius}" length="${wheel_thickness}"/>
-        </geometry>
-        <material name="red" />
-      </visual>
-      <collision>
-        <origin xyz="0 0 0" rpy="0 0 0"/>
-        <geometry>
-          <cylinder radius="${wheel_radius}" length="${wheel_thickness}"/>
-        </geometry>
-      </collision>
-      <xacro:solid_cylinder_inertial
-          rpy="0 0 0" xyz="0 0 0"
-          mass="${wheel_mass}"
-          radius="${wheel_radius}" length="${wheel_thickness}" />
-    </link>
-    <joint name="${name}_wheel_joint" type="continuous">
-      <parent link="${name}_steer_link"/>
-      <child link="${name}_wheel_link"/>
-      <origin xyz="0 0 ${-steer_height}" rpy="${-90 * deg_to_rad} 0 0"/>
-      <axis xyz="0 0 1"/>
-    </joint>
-    <transmission name="${name}_steer_joint_trans">
-      <type>transmission_interface/SimpleTransmission</type>
-      <actuator name="${name}_steer_joint_motor">
-        <mechanicalReduction>1</mechanicalReduction>
-        <hardwareInterface>hardware_interface/PositionJointInterface</hardwareInterface>
-      </actuator>
-      <joint name="${name}_steer_joint">
-        <hardwareInterface>hardware_interface/PositionJointInterface</hardwareInterface>
-      </joint>
-    </transmission>
-    <transmission name="${name}_wheel_joint_trans">
-      <type>transmission_interface/SimpleTransmission</type>
-      <actuator name="${name}_wheel_joint_motor">
-        <mechanicalReduction>1</mechanicalReduction>
-        <hardwareInterface>hardware_interface/VelocityJointInterface</hardwareInterface>
-      </actuator>
-      <joint name="${name}_wheel_joint">
-        <hardwareInterface>hardware_interface/VelocityJointInterface</hardwareInterface>
-      </joint>
-    </transmission>
-    <gazebo reference="${name}_steer_link">
-      <material>Gazebo/Blue</material>
-    </gazebo>
-    <gazebo reference="${name}_wheel_link">
-      <material>Gazebo/Red</material>
-    </gazebo>
-  </xacro:macro>
-  <!-- Bicycle model rear wheel link (required for steer_drive_controller) -->
-  <xacro:macro name="rear_wheel"
-    params="
-      name
-      parent
-      wheel_radius
-      wheel_thickness
-      wheel_mass
-      *origin">
-    <link name="${name}_wheel_link">
-      <visual>
-        <origin xyz="0 0 0" rpy="0 0 0"/>
-        <geometry>
-          <cylinder radius="${wheel_radius}" length="${wheel_thickness}"/>
-        </geometry>
-        <material name="yellow" />
-      </visual>
-      <collision>
-        <origin xyz="0 0 0" rpy="0 0 0"/>
-        <geometry>
-          <cylinder radius="${wheel_radius}" length="${wheel_thickness}"/>
-        </geometry>
-      </collision>
-      <xacro:solid_cylinder_inertial
-          rpy="0 0 0" xyz="0 0 0"
-          mass="${wheel_mass}"
-          radius="${wheel_radius}" length="${wheel_thickness}" />
-    </link>
-    <joint name="${name}_wheel_joint" type="continuous">
-      <parent link="${parent}_link"/>
-      <child link="${name}_wheel_link"/>
-      <xacro:insert_block name="origin"/>
-      <axis xyz="0 0 1"/>
-    </joint>
-    <transmission name="${name}_wheel_joint_trans">
-      <type>transmission_interface/SimpleTransmission</type>
-      <actuator name="${name}_wheel_joint_motor">
-        <mechanicalReduction>1</mechanicalReduction>
-        <hardwareInterface>hardware_interface/VelocityJointInterface</hardwareInterface>
-      </actuator>
-      <joint name="${name}_wheel_joint">
-        <hardwareInterface>hardware_interface/VelocityJointInterface</hardwareInterface>
-      </joint>
-    </transmission>
-    <gazebo reference="${name}_wheel_link">
-      <material>Gazebo/Yellow</material>
-    </gazebo>
-  </xacro:macro>
-  <!-- Bicycle model front wheel link (passive - no transmission) -->
-  <xacro:macro name="front_wheel"
-    params="
-      name
-      parent
-      wheel_radius
-      wheel_thickness
-      wheel_mass
-      *origin">
-    <link name="${name}_wheel_link">
-      <visual>
-        <origin xyz="0 0 0" rpy="0 0 0"/>
-        <geometry>
-          <cylinder radius="${wheel_radius}" length="${wheel_thickness}"/>
-        </geometry>
-        <material name="yellow" />
-      </visual>
-      <collision>
-        <origin xyz="0 0 0" rpy="0 0 0"/>
-        <geometry>
-          <cylinder radius="${wheel_radius}" length="${wheel_thickness}"/>
-        </geometry>
-      </collision>
-      <xacro:solid_cylinder_inertial
-          rpy="0 0 0" xyz="0 0 0"
-          mass="${wheel_mass}"
-          radius="${wheel_radius}" length="${wheel_thickness}" />
-    </link>
-    <joint name="${name}_wheel_joint" type="continuous">
-      <parent link="${parent}_link"/>
-      <child link="${name}_wheel_link"/>
-      <xacro:insert_block name="origin"/>
-      <axis xyz="0 0 1"/>
-    </joint>
-    <gazebo reference="${name}_wheel_link">
-      <material>Gazebo/Yellow</material>
-    </gazebo>
-    <gazebo reference="${name}_wheel_joint">
-      <provideFeedback>true</provideFeedback>
-    </gazebo>
-  </xacro:macro>
-  <!-- Car steering model rear wheel links (left/right) -->
-  <xacro:macro name="rear_wheel_lr"
-    params="
-      name
-      parent
-      wheel_radius
-      wheel_thickness
-      wheel_mass
-      *origin">
-    <link name="${name}_wheel_link">
-      <visual>
-        <origin xyz="0 0 0" rpy="0 0 0"/>
-        <geometry>
-          <cylinder radius="${wheel_radius}" length="${wheel_thickness}"/>
-        </geometry>
-        <material name="red" />
-      </visual>
-      <collision>
-        <origin xyz="0 0 0" rpy="0 0 0"/>
-        <geometry>
-          <cylinder radius="${wheel_radius}" length="${wheel_thickness}"/>
-        </geometry>
-      </collision>
-      <xacro:solid_cylinder_inertial
-          rpy="0 0 0" xyz="0 0 0"
-          mass="${wheel_mass}"
-          radius="${wheel_radius}" length="${wheel_thickness}" />
-    </link>
-    <joint name="${name}_wheel_joint" type="continuous">
-      <parent link="${parent}_link"/>
-      <child link="${name}_wheel_link"/>
-      <xacro:insert_block name="origin"/>
-      <axis xyz="0 0 1"/>
-    </joint>
-    <transmission name="${name}_wheel_joint_trans">
-      <type>transmission_interface/SimpleTransmission</type>
-      <actuator name="${name}_wheel_joint_motor">
-        <mechanicalReduction>1</mechanicalReduction>
-        <hardwareInterface>hardware_interface/VelocityJointInterface</hardwareInterface>
-      </actuator>
-      <joint name="${name}_wheel_joint">
-        <hardwareInterface>hardware_interface/VelocityJointInterface</hardwareInterface>
-      </joint>
-    </transmission>
-    <gazebo reference="${name}_wheel_link">
-      <material>Gazebo/Red</material>
-    </gazebo>
-  </xacro:macro>
+    </xacro:macro>
 </robot>

Commit message: noetic ackermann implemented (not what expected)

File: src/description_bauda_akm/description/robot.urdf.xacro (robot description, xacro)
@@ -3,4 +3,4 @@
     <xacro:include filename="robot_core.xacro" />
     <!-- <xacro:include filename="gazebo_control.xacro" /> -->
-    <xacro:include filename="ros2_control.xacro" />
+    <xacro:include filename="ros_control.xacro" />
 </robot>

File: src/description_bauda_akm/description/robot_core.xacro (robot description, xacro)
@@ -5,5 +5,5 @@
     <!-- Define robot constants https://navigation.ros.org/setup_guides/urdf/setup_urdf.html -->
     <xacro:property name="yaml_file" value="$(find description_bauda_akm)/config/vehicle.yaml" />
-    <xacro:property name="vehicle_dict" value="${load_yaml(yaml_file)}"/>
+    <xacro:property name="vehicle_dict" value="${xacro.load_yaml(yaml_file)}"/>
     <xacro:property name="base_mass" value="${vehicle_dict['base']['mass']}" />
     <xacro:property name="base_length" value="${vehicle_dict['base']['length']}" />
@@ -174,9 +174,8 @@
     </gazebo> -->
     <!-- FRONT LEFT WHEEL -->
-    <joint name="front_left_wheel_joint" type="continuous">
+    <joint name="front_left_wheel_joint" type="fixed">
         <parent link="left_steering_link"/>
         <child link="front_left_wheel"/>
         <origin xyz="0 0 0" rpy="-${pi/2} 0 0" />
-        <axis xyz="0 0 1"/>
     </joint>
     <link name="front_left_wheel">
@@ -200,9 +199,8 @@
     </gazebo>
     <!-- FRONT RIGHT WHEEL -->
-    <joint name="front_right_wheel_joint" type="continuous">
+    <joint name="front_right_wheel_joint" type="fixed">
         <parent link="right_steering_link"/>
         <child link="front_right_wheel"/>
         <origin xyz="0 0 0" rpy="${pi/2} 0 0" />
-        <axis xyz="0 0 -1"/>
     </joint>
     <link name="front_right_wheel">
@@ -225,5 +223,5 @@
         <material>Gazebo/Blue</material>
     </gazebo>
-    <!-- STEERING WHEEL -->
+    <!-- STEERING WHEEL
     <joint name="steering_wheel_joint" type="continuous">
         <parent link="base_link"/>
@@ -250,4 +248,4 @@
     <gazebo reference="steering_wheel">
         <material>Gazebo/Blue</material>
-    </gazebo>
+    </gazebo> -->
  </robot>
