Commit message: 3D_lidar

File: src/description_bauda_akm/description/2D_lidar.xacro (robot description, xacro)
@@ -1,8 +1,13 @@
 <?xml version="1.0"?>
 <robot xmlns:xacro="http://www.ros.org/wiki/xacro"  name="bauda_diff">
-    <joint name="laser_joit" type="fixed">
+    <xacro:property name="yaml_file" value="$(find description_bauda_akm)/config/vehicle.yaml" />
+    <xacro:property name="vehicle_dict" value="${xacro.load_yaml(yaml_file)}"/>
+    <xacro:property name="lidar_x" value="${vehicle_dict['lidar']['x']}" />
+    <xacro:property name="lidar_y" value="${vehicle_dict['lidar']['y']}" />
+    <xacro:property name="lidar_z" value="${vehicle_dict['lidar']['z']}" />
+    <joint name="laser_joint" type="fixed">
         <parent link="chassis"/>
         <child link="laser_frame"/>
-        <origin xyz="0.1 0 0.175" rpy="0 0 0"/>
+        <origin xyz="${lidar_x} ${lidar_y} ${lidar_z}" rpy="0 0 0"/>
     </joint>
     <link name="laser_frame">
@@ -26,5 +31,5 @@
         <sensor name="laser" type="ray">
             <pose> 0 0 0 0 0 0 </pose>
-            <visualize>false</visualize>
+            <visualize>true</visualize>
             <update_rate>10</update_rate>
             <ray>

File: src/description_bauda_akm/description/camera.xacro (robot description, xacro)
@@ -1,8 +1,13 @@
 <?xml version="1.0"?>
 <robot xmlns:xacro="http://www.ros.org/wiki/xacro"  name="bauda_diff">
-    <joint name="camera_joit" type="fixed">
+    <xacro:property name="yaml_file" value="$(find description_bauda_akm)/config/vehicle.yaml" />
+    <xacro:property name="vehicle_dict" value="${xacro.load_yaml(yaml_file)}"/>
+    <xacro:property name="camera_x" value="${vehicle_dict['camera']['x']}" />
+    <xacro:property name="camera_y" value="${vehicle_dict['camera']['y']}" />
+    <xacro:property name="camera_z" value="${vehicle_dict['camera']['z']}" />
+    <joint name="camera_joint" type="fixed">
         <parent link="chassis"/>
         <child link="camera_link"/>
-        <origin xyz="0.305 0 0.08" rpy="0 0 0"/>
+        <origin xyz="${camera_x} ${camera_y} ${camera_z}" rpy="0 0 0"/>
     </joint>
     <link name="camera_link">
@@ -24,5 +29,5 @@
         <sensor name="camera" type="camera">
             <pose> 0 0 0 0 0 0 </pose>
-            <visualize>false</visualize>
+            <visualize>true</visualize>
             <update_rate>10</update_rate>
             <camera>
@@ -38,5 +43,5 @@
                 </clip>
             </camera>
-            <plugin name="laser_controller" filename="libgazebo_ros_camera.so">
+            <plugin name="camera_controller" filename="libgazebo_ros_camera.so">
                 <frame_name>camera_link_optical</frame_name>
             </plugin>

File: src/description_bauda_akm/description/depth_camera.xacro (robot description, xacro)
@@ -1,8 +1,13 @@
 <?xml version="1.0"?>
 <robot xmlns:xacro="http://www.ros.org/wiki/xacro"  name="bauda_diff">
-    <joint name="camera_joit" type="fixed">
+    <xacro:property name="yaml_file" value="$(find description_bauda_akm)/config/vehicle.yaml" />
+    <xacro:property name="vehicle_dict" value="${xacro.load_yaml(yaml_file)}"/>
+    <xacro:property name="camera_x" value="${vehicle_dict['camera']['x']}" />
+    <xacro:property name="camera_y" value="${vehicle_dict['camera']['y']}" />
+    <xacro:property name="camera_z" value="${vehicle_dict['camera']['z']}" />
+    <joint name="camera_joint" type="fixed">
         <parent link="chassis"/>
         <child link="camera_link"/>
-        <origin xyz="0.305 0 0.08" rpy="0 0 0"/>
+        <origin xyz="${camera_x} ${camera_y} ${camera_z}" rpy="0 0 0"/>
     </joint>
     <link name="camera_link">
@@ -20,9 +25,9 @@
     </joint>
     <link name="camera_link_optical"/>
-   <gazebo reference="camera_link">
+    <gazebo reference="camera_link">
         <material>Gazebo/Red</material>
         <sensor name="camera" type="depth">
             <pose> 0 0 0 0 0 0 </pose>
-            <visualize>false</visualize>
+            <visualize>true</visualize>
             <update_rate>10</update_rate>
             <camera>
@@ -38,5 +43,5 @@
                 </clip>
             </camera>
-            <plugin name="laser_controller" filename="libgazebo_ros_camera.so">
+            <plugin name="depth_camera_controller" filename="libgazebo_ros_camera.so">
                 <frame_name>camera_link_optical</frame_name>
                 <min_depth>0.1</min_depth>

File: src/description_bauda_akm/description/robot.urdf.xacro (robot description, xacro)
@@ -2,5 +2,8 @@
 <robot xmlns:xacro="http://www.ros.org/wiki/xacro"  name="bauda_diff">
     <xacro:include filename="robot_core.xacro" />
-    <!-- <xacro:include filename="gazebo_control.xacro" /> -->
     <xacro:include filename="ros2_control.xacro" />
+    <!-- <xacro:include filename="depth_camera.xacro" /> -->
+    <xacro:include filename="camera.xacro" />
+    <!-- <xacro:include filename="2D_lidar.xacro" /> -->
+    <xacro:include filename="3D_lidar.xacro" />
 </robot>

File: src/description_bauda_akm/description/robot_core.xacro (robot description, xacro)
@@ -5,5 +5,5 @@
     <!-- Define robot constants https://navigation.ros.org/setup_guides/urdf/setup_urdf.html -->
     <xacro:property name="yaml_file" value="$(find description_bauda_akm)/config/vehicle.yaml" />
-    <xacro:property name="vehicle_dict" value="${load_yaml(yaml_file)}"/>
+    <xacro:property name="vehicle_dict" value="${xacro.load_yaml(yaml_file)}"/>
     <xacro:property name="base_mass" value="${vehicle_dict['base']['mass']}" />
     <xacro:property name="base_length" value="${vehicle_dict['base']['length']}" />
@@ -122,22 +122,5 @@
             <inertia ixx="0.002" ixy="0" ixz="0" iyy="0.002" iyz="0" izz="0.002"/>
         </inertial>
-        <!-- <visual>
-            <geometry>
-                <cylinder radius="0.001" length="0.001"/>
-            </geometry>
-            <material name="blue"/>
-        </visual>
-        <collision>
-            <geometry>
-                <cylinder radius="0.001" length="0.001"/>
-            </geometry>
-        </collision>
-        <xacro:inertial_cylinder mass="0.001" length="0.001" radius="0.001">
-            <origin xyz="0 0 0" rpy="0 0 0"/>
-        </xacro:inertial_cylinder> -->
     </link>
-    <!-- <gazebo reference="rear_right_wheel">
-        <material>Gazebo/Blue</material>
-    </gazebo> -->
     <!-- RIGHT STEERING -->
     <joint name="right_steering_joint" type="revolute">
@@ -155,22 +138,5 @@
             <inertia ixx="0.002" ixy="0" ixz="0" iyy="0.002" iyz="0" izz="0.002"/>
         </inertial>
-        <!-- <visual>
-            <geometry>
-                <cylinder radius="0.001" length="0.001"/>
-            </geometry>
-            <material name="blue"/>
-        </visual>
-        <collision>
-            <geometry>
-                <cylinder radius="0.001" length="0.001"/>
-            </geometry>
-        </collision>
-        <xacro:inertial_cylinder mass="0.001" length="0.001" radius="0.001">
-            <origin xyz="0 0 0" rpy="0 0 0"/>
-        </xacro:inertial_cylinder> -->
     </link>
-    <!-- <gazebo reference="rear_right_wheel">
-        <material>Gazebo/Blue</material>
-    </gazebo> -->
     <!-- FRONT LEFT WHEEL -->
     <joint name="front_left_wheel_joint" type="continuous">
@@ -225,29 +191,3 @@
         <material>Gazebo/Blue</material>
     </gazebo>
-    <!-- STEERING WHEEL -->
-    <joint name="steering_wheel_joint" type="continuous">
-        <parent link="base_link"/>
-        <child link="steering_wheel"/>
-        <origin xyz="${wheel_distance_between_axes} 0 ${base_height + 2 * wheel_radius}" rpy="0 0 0"/>
-        <axis xyz="0 0 1"/>
-    </joint>
-    <link name="steering_wheel">
-        <visual>
-            <geometry>
-                <cylinder radius="${wheel_radius}" length="${wheel_width}"/>
-            </geometry>
-            <material name="blue"/>
-        </visual>
-        <collision>
-            <geometry>
-                <cylinder radius="${wheel_radius}" length="${wheel_width}"/>
-            </geometry>
-        </collision>
-        <xacro:inertial_cylinder mass="${wheel_mass}" length="${wheel_width}" radius="${wheel_radius}">
-            <origin xyz="0 0 0" rpy="0 0 0"/>
-        </xacro:inertial_cylinder>
-    </link>
-    <gazebo reference="steering_wheel">
-        <material>Gazebo/Blue</material>
-    </gazebo>
  </robot>

File: src/description_bauda_akm/description/ros2_control.xacro (robot description, xacro)
@@ -7,29 +7,9 @@
         </hardware>
         <joint name="rear_left_wheel_joint">
-            <command_interface name="velocity">
-                <param name="min">-10</param>
-                <param name="max">10</param>
-            </command_interface>
+            <command_interface name="velocity"/>
             <state_interface name="velocity"/>
         </joint>
         <joint name="rear_right_wheel_joint">
-            <command_interface name="velocity">
-                <param name="min">-10</param>
-                <param name="max">10</param>
-            </command_interface>
-            <state_interface name="velocity"/>
-        </joint>
-        <joint name="front_left_wheel_joint">
-            <command_interface name="velocity">
-                <param name="min">-10</param>
-                <param name="max">10</param>
-            </command_interface>
-            <state_interface name="velocity"/>
-        </joint>
-        <joint name="front_right_wheel_joint">
-            <command_interface name="velocity">
-                <param name="min">-10</param>
-                <param name="max">10</param>
-            </command_interface>
+            <command_interface name="velocity"/>
             <state_interface name="velocity"/>
         </joint>
@@ -48,11 +28,4 @@
             <state_interface name="position"/>
         </joint>
-        <joint name="steering_wheel_joint">
-            <command_interface name="position">
-                <param name="min">${-steering_limit_angle}</param>
-                <param name="max">${steering_limit_angle}</param>
-            </command_interface>
-            <state_interface name="position"/>
-        </joint>
     </ros2_control>
     <gazebo>
