Commit message: velodyne

File: src/description_bauda_akm/description/2D_lidar.xacro (robot description, xacro)
@@ -1,9 +1,4 @@
 <?xml version="1.0"?>
 <robot xmlns:xacro="http://www.ros.org/wiki/xacro"  name="bauda_diff">
-    <xacro:property name="yaml_file" value="$(find description_bauda_akm)/config/vehicle.yaml" />
-    <xacro:property name="vehicle_dict" value="${xacro.load_yaml(yaml_file)}"/>
-    <xacro:property name="lidar_x" value="${vehicle_dict['lidar']['x']}" />
-    <xacro:property name="lidar_y" value="${vehicle_dict['lidar']['y']}" />
-    <xacro:property name="lidar_z" value="${vehicle_dict['lidar']['z']}" />
     <joint name="laser_joint" type="fixed">
         <parent link="chassis"/>
@@ -48,5 +43,5 @@
             <plugin name="laser_controller" filename="libgazebo_ros_ray_sensor.so">
                 <ros>
-                    <argument>~/out:=scan</argument>
+                    <argument>--ros-args -r ~/out:=/scan</argument>
                 </ros>
                 <output_type>sensor_msgs/LaserScan</output_type>

File: src/description_bauda_akm/description/camera.xacro (robot description, xacro)
@@ -1,9 +1,4 @@
 <?xml version="1.0"?>
 <robot xmlns:xacro="http://www.ros.org/wiki/xacro"  name="bauda_diff">
-    <xacro:property name="yaml_file" value="$(find description_bauda_akm)/config/vehicle.yaml" />
-    <xacro:property name="vehicle_dict" value="${xacro.load_yaml(yaml_file)}"/>
-    <xacro:property name="camera_x" value="${vehicle_dict['camera']['x']}" />
-    <xacro:property name="camera_y" value="${vehicle_dict['camera']['y']}" />
-    <xacro:property name="camera_z" value="${vehicle_dict['camera']['z']}" />
     <joint name="camera_joint" type="fixed">
         <parent link="chassis"/>
@@ -25,5 +20,5 @@
     </joint>
     <link name="camera_link_optical"/>
-   <gazebo reference="camera_link">
+    <gazebo reference="camera_link">
         <material>Gazebo/Red</material>
         <sensor name="camera" type="camera">

File: src/description_bauda_akm/description/depth_camera.xacro (robot description, xacro)
@@ -1,9 +1,4 @@
 <?xml version="1.0"?>
 <robot xmlns:xacro="http://www.ros.org/wiki/xacro"  name="bauda_diff">
-    <xacro:property name="yaml_file" value="$(find description_bauda_akm)/config/vehicle.yaml" />
-    <xacro:property name="vehicle_dict" value="${xacro.load_yaml(yaml_file)}"/>
-    <xacro:property name="camera_x" value="${vehicle_dict['camera']['x']}" />
-    <xacro:property name="camera_y" value="${vehicle_dict['camera']['y']}" />
-    <xacro:property name="camera_z" value="${vehicle_dict['camera']['z']}" />
     <joint name="camera_joint" type="fixed">
         <parent link="chassis"/>

File: src/description_bauda_akm/description/robot.urdf.xacro (robot description, xacro)
@@ -1,4 +1,35 @@
 <?xml version="1.0"?>
 <robot xmlns:xacro="http://www.ros.org/wiki/xacro"  name="bauda_diff">
+    <!-- Define robot constants https://navigation.ros.org/setup_guides/urdf/setup_urdf.html -->
+    <xacro:property name="yaml_file" value="$(find description_bauda_akm)/config/vehicle.yaml" />
+    <xacro:property name="vehicle_dict" value="${xacro.load_yaml(yaml_file)}"/>
+    <xacro:property name="base_mass" value="${vehicle_dict['base']['mass']}" />
+    <xacro:property name="base_length" value="${vehicle_dict['base']['length']}" />
+    <xacro:property name="base_width" value="${vehicle_dict['base']['width']}" />
+    <xacro:property name="base_height" value="${vehicle_dict['base']['height']}" />
+    <xacro:property name="wheel_mass" value="${vehicle_dict['wheel']['mass']}" />
+    <xacro:property name="wheel_radius" value="${vehicle_dict['wheel']['radius']}" />
+    <xacro:property name="wheel_width" value="${vehicle_dict['wheel']['width']}" />
+    <xacro:property name="wheel_ygap" value="${vehicle_dict['wheel']['ygap']}" />
+    <xacro:property name="wheel_rear_xoff" value="${vehicle_dict['wheel']['rear_xoff']}" />
+    <xacro:property name="wheel_distance_between_axes" value="${vehicle_dict['wheel']['distance_between_axes']}" />
+    <xacro:property name="steering_limit_angle" value="${vehicle_dict['steering']['limit_angle']}" />
+    <xacro:property name="steering_limit_effort" value="${vehicle_dict['steering']['limit_effort']}" />
+    <xacro:property name="steering_limit_velocity" value="${vehicle_dict['steering']['limit_velocity']}" />
+    <xacro:property name="lidar_x" value="${vehicle_dict['lidar']['x']}" />
+    <xacro:property name="lidar_y" value="${vehicle_dict['lidar']['y']}" />
+    <xacro:property name="lidar_z" value="${vehicle_dict['lidar']['z']}" />
+    <xacro:property name="camera_x" value="${vehicle_dict['camera']['x']}" />
+    <xacro:property name="camera_y" value="${vehicle_dict['camera']['y']}" />
+    <xacro:property name="camera_z" value="${vehicle_dict['camera']['z']}" />
+    <xacro:property name="lidar_x" value="${vehicle_dict['camera']['x']}" />
+    <xacro:property name="lidar_y" value="${vehicle_dict['lidar']['y']}" />
+    <xacro:property name="lidar_z" value="${vehicle_dict['lidar']['z']}" />
+    <xacro:property name="lidar_organize_cloud" value="${vehicle_dict['lidar']['organize_cloud']}" />
+    <xacro:property name="lidar_frequency" value="${vehicle_dict['lidar']['frequency']}" />
+    <xacro:property name="lidar_samples" value="${vehicle_dict['lidar']['samples']}" />
+    <xacro:property name="lidar_gpu" value="${vehicle_dict['lidar']['gpu']}" />
+    <xacro:include filename="inertials.xacro" />
+    <xacro:include filename="materials.xacro" />
     <xacro:include filename="robot_core.xacro" />
     <xacro:include filename="ros2_control.xacro" />
@@ -6,4 +37,5 @@
     <xacro:include filename="camera.xacro" />
     <!-- <xacro:include filename="2D_lidar.xacro" /> -->
-    <xacro:include filename="3D_lidar.xacro" />
+    <!-- <xacro:include filename="VLP-16.urdf.xacro" /> -->
+    <xacro:include filename="HDL-32E.urdf.xacro" />
 </robot>

File: src/description_bauda_akm/description/robot_core.xacro (robot description, xacro)
@@ -1,22 +1,4 @@
 <?xml version="1.0"?>
 <robot xmlns:xacro="http://www.ros.org/wiki/xacro" >
-    <xacro:include filename="inertials.xacro"/>
-    <xacro:include filename="materials.xacro"/>
-    <!-- Define robot constants https://navigation.ros.org/setup_guides/urdf/setup_urdf.html -->
-    <xacro:property name="yaml_file" value="$(find description_bauda_akm)/config/vehicle.yaml" />
-    <xacro:property name="vehicle_dict" value="${xacro.load_yaml(yaml_file)}"/>
-    <xacro:property name="base_mass" value="${vehicle_dict['base']['mass']}" />
-    <xacro:property name="base_length" value="${vehicle_dict['base']['length']}" />
-    <xacro:property name="base_width" value="${vehicle_dict['base']['width']}" />
-    <xacro:property name="base_height" value="${vehicle_dict['base']['height']}" />
-    <xacro:property name="wheel_mass" value="${vehicle_dict['wheel']['mass']}" />
-    <xacro:property name="wheel_radius" value="${vehicle_dict['wheel']['radius']}" />
-    <xacro:property name="wheel_width" value="${vehicle_dict['wheel']['width']}" />
-    <xacro:property name="wheel_ygap" value="${vehicle_dict['wheel']['ygap']}" />
-    <xacro:property name="wheel_rear_xoff" value="${vehicle_dict['wheel']['rear_xoff']}" />
-    <xacro:property name="wheel_distance_between_axes" value="${vehicle_dict['wheel']['distance_between_axes']}" />
-    <xacro:property name="steering_limit_angle" value="${vehicle_dict['steering']['limit_angle']}" />
-    <xacro:property name="steering_limit_effort" value="${vehicle_dict['steering']['limit_effort']}" />
-    <xacro:property name="steering_limit_velocity" value="${vehicle_dict['steering']['limit_velocity']}" />
     <!-- BASE LINK -->
     <link name="base_link" />

File: src/description_bauda_akm/description/ros2_control.xacro (robot description, xacro)
@@ -1,5 +1,4 @@
 <?xml version="1.0"?>
 <robot xmlns:xacro="http://www.ros.org/wiki/xacro">
-    <xacro:property name="steering_limit_angle" value="${vehicle_dict['steering']['limit_angle']}" />
     <ros2_control name="GazeboSystem" type="system">
         <hardware>
@@ -8,8 +7,10 @@
         <joint name="rear_left_wheel_joint">
             <command_interface name="velocity"/>
+            <state_interface name="position"/>
             <state_interface name="velocity"/>
         </joint>
         <joint name="rear_right_wheel_joint">
             <command_interface name="velocity"/>
+            <state_interface name="position"/>
             <state_interface name="velocity"/>
         </joint>
@@ -28,4 +29,17 @@
             <state_interface name="position"/>
         </joint>
+        <joint name="front_right_wheel_joint">
+            <state_interface name="position"/>
+            <state_interface name="velocity"/>
+        </joint>
+        <joint name="front_left_wheel_joint">
+            <state_interface name="position"/>
+            <state_interface name="velocity"/>
+        </joint>
+        <joint name="lidar_joint">
+            <command_interface name="velocity"/>
+            <state_interface name="position"/>
+            <state_interface name="velocity"/>
+        </joint>
     </ros2_control>
     <gazebo>

File: src/description_bauda_akm/description/velodyne.xacro (robot description, xacro)
@@ -1,59 +1,44 @@
 <?xml version="1.0"?>
 <robot xmlns:xacro="http://www.ros.org/wiki/xacro"  name="bauda_diff">
-    <xacro:property name="yaml_file" value="$(find description_bauda_akm)/config/vehicle.yaml" />
-    <xacro:property name="vehicle_dict" value="${xacro.load_yaml(yaml_file)}"/>
-    <xacro:property name="lidar_x" value="${vehicle_dict['lidar']['x']}" />
-    <xacro:property name="lidar_y" value="${vehicle_dict['lidar']['y']}" />
-    <xacro:property name="lidar_z" value="${vehicle_dict['lidar']['z']}" />
     <joint name="base_lidar_joint" type="fixed">
         <parent link="chassis"/>
         <child link="lidar_base"/>
-        <origin xyz="${lidar_x} ${lidar_y} ${lidar_z}" rpy="0 0 0"/>
+        <origin xyz="${lidar_x} ${lidar_y} ${lidar_z + lidar_base_height / 2}" rpy="0 0 0"/>
     </joint>
     <link name="lidar_base">
         <visual>
-            <!-- <origin xyz="0 0 0.029335"/> -->
             <geometry>
-                <cylinder radius="0.04267" length="0.05867"/>
+                <cylinder radius="${lidar_radius}" length="${lidar_base_height}"/>
             </geometry>
         </visual>
         <collision>
-            <!-- <origin xyz="0 0 0.029335"/> -->
             <geometry>
-                <cylinder radius="0.04267" length="0.05867"/>
+                <cylinder radius="${lidar_radius}" length="${lidar_base_height}"/>
             </geometry>
         </collision>
-        <inertial>
-            <mass value="1.2" />
-            <inertia ixx="0.001087473" ixy="0.0" ixz="0.0"
-                    iyy="0.001087473" iyz="0.0"
-                    izz="0.001092437" />
-        </inertial>
+        <xacro:inertial_cylinder mass="${lidar_mass}" length="${lidar_base_height}" radius="${lidar_radius}">
+            <origin xyz="0 0 0" rpy="0 0 0"/>
+        </xacro:inertial_cylinder>
     </link>
     <joint name="lidar_joint" type="continuous">
         <parent link="lidar_base"/>
         <child link="laser_frame"/>
-        <origin xyz="0 0 0.05867" rpy="0 0 0" />
+        <origin xyz="0 0 ${lidar_base_height / 2 + lidar_top_height / 2}" rpy="0 0 0" />
         <axis xyz="0 0 1"/>
     </joint>
     <link name="laser_frame">
         <visual>
-            <!-- <origin xyz="0 0 0.095455"/> -->
             <geometry>
-                <cylinder radius="0.04267" length="0.07357"/>
+                <cylinder radius="${lidar_radius}" length="${lidar_top_height}"/>
             </geometry>
         </visual>
-        <!-- <collision>
-            <origin xyz="0 0 0.095455"/>
+        <collision>
             <geometry>
-                <cylinder radius="0.04267" length="0.07357"/>
+                <cylinder radius="${lidar_radius}" length="${lidar_top_height}"/>
             </geometry>
-        </collision> -->
-        <inertial>
-            <mass value="1.2" />
-            <inertia ixx="0.000090623" ixy="0.0" ixz="0.0"
-                    iyy="0.000090623" iyz="0.0"
-                    izz="0.000091036" />
-        </inertial>
+        </collision>
+        <xacro:inertial_cylinder mass="${lidar_mass}" length="${lidar_top_height}" radius="${lidar_radius}">
+            <origin xyz="0 0 0" rpy="0 0 0"/>
+        </xacro:inertial_cylinder>
     </link>
     <gazebo reference="laser_frame">
@@ -64,19 +49,19 @@
             <update_rate>10</update_rate>
             <ray>
-                <noise>
+                <!-- <noise>
                     <type>gaussian</type>
                     <mean>0.0</mean>
                     <stddev>0.02</stddev>
-                </noise>
+                </noise> -->
                 <scan>
-                    <horizontal>
+                    <vertical>
                         <samples>32</samples>
                         <resolution>1</resolution>
                         <min_angle>-0.53529248</min_angle>
                         <max_angle>0.18622663</max_angle>
-                    </horizontal>
+                    </vertical>
                 </scan>
                 <range>
-                    <min>0.05</min>
+                    <min>0.06</min>
                     <max>70</max>
                     <resolution>0.02</resolution>
@@ -85,7 +70,7 @@
             <plugin name="laser_controller" filename="libgazebo_ros_ray_sensor.so">
                 <ros>
-                    <argument>~/out:=scan</argument>
+                    <argument>--ros-args -r ~/out:=/scan</argument>
                 </ros>
-                <output_type>sensor_msgs/LaserScan</output_type>
+                <output_type>sensor_msgs/PointCloud2</output_type>
                 <frame_name>laser_frame</frame_name>
             </plugin>

Commit message: ackermann joystick teleop

File: src/description_bauda_akm/description/2D_lidar.xacro (robot description, xacro)
@@ -1,10 +1,10 @@
 <?xml version="1.0"?>
 <robot xmlns:xacro="http://www.ros.org/wiki/xacro"  name="bauda_diff">
-    <joint name="laser_joint" type="fixed">
+    <joint name="laser_base_joint" type="fixed">
         <parent link="chassis"/>
-        <child link="laser_frame"/>
+        <child link="lidar_base"/>
         <origin xyz="${lidar_x} ${lidar_y} ${lidar_z}" rpy="0 0 0"/>
     </joint>
-    <link name="laser_frame">
+    <link name="lidar_base">
         <visual>
             <geometry>
@@ -21,4 +21,11 @@
             <origin xyz="0 0 0" rpy="0 0 0"/>
         </xacro:inertial_cylinder>
+    </link>
+    <joint name="laser_frame_joint" type="fixed">
+        <parent link="lidar_base" />
+        <child link="laser_frame" />
+        <origin xyz="0 0 0.005" rpy="0 0 0"/>
+    </joint>
+    <link name="laser_frame">
     </link>
    <gazebo reference="laser_frame">

File: src/description_bauda_akm/description/robot.urdf.xacro (robot description, xacro)
@@ -23,5 +23,5 @@
     <xacro:property name="camera_y" value="${vehicle_dict['camera']['y']}" />
     <xacro:property name="camera_z" value="${vehicle_dict['camera']['z']}" />
-    <xacro:property name="lidar_x" value="${vehicle_dict['camera']['x']}" />
+    <xacro:property name="lidar_x" value="${vehicle_dict['lidar']['x']}" />
     <xacro:property name="lidar_y" value="${vehicle_dict['lidar']['y']}" />
     <xacro:property name="lidar_z" value="${vehicle_dict['lidar']['z']}" />
@@ -36,6 +36,6 @@
     <!-- <xacro:include filename="depth_camera.xacro" /> -->
     <xacro:include filename="camera.xacro" />
-    <!-- <xacro:include filename="2D_lidar.xacro" /> -->
+    <xacro:include filename="2D_lidar.xacro" />
     <!-- <xacro:include filename="VLP-16.urdf.xacro" /> -->
-    <xacro:include filename="HDL-32E.urdf.xacro" />
+    <!-- <xacro:include filename="HDL-32E.urdf.xacro" /> -->
 </robot>
